Commit message: modificaciones para multiples robots

File: src/diffdrive_description/urdf/mobile_base.xacro (robot description, xacro)
@@ -1,4 +1,5 @@
 <?xml version="1.0"?>
 <robot xmlns:xacro="http://www.ros.org/wiki/xacro">
+    <xacro:property name="tf_prefix" value=""/>
     <xacro:property name="base_length" value="0.23"/> <!-- Largo del chasis [m]-->
     <xacro:property name="base_width" value="0.15"/>  <!-- Ancho del chasis [m]-->
@@ -7,5 +8,5 @@
     <xacro:property name="wheel_length" value="0.03"/> <!-- Grosor de ruedas [m]-->
     <xacro:property name="caster_radius" value="0.009525"/>
-    <link name="base_footprint"/>
+    <link name="${tf_prefix}base_footprint"/>
     <!-- CHASIS PRINCIPAL -->
     <!--base_link
@@ -13,5 +14,5 @@
         Ubicación Centro geométrico del chasis
     -->
-    <link name="base_link">
+    <link name="${tf_prefix}base_link">
         <visual>
             <geometry>
@@ -48,8 +49,8 @@
         </link>
     </xacro:macro>
-    <xacro:wheel_link prefix="left"/>
-    <xacro:wheel_link prefix="right"/>
+    <xacro:wheel_link prefix="${tf_prefix}left"/>
+    <xacro:wheel_link prefix="${tf_prefix}right"/>
     <!-- RUEDA LOCA -->
-    <link name="caster_wheel_link">
+    <link name="${tf_prefix}caster_wheel_link">
         <visual>
             <geometry>
@@ -68,5 +69,5 @@
     </link>
     <!-- IMU Link -->
-    <link name="imu_link">
+    <link name="${tf_prefix}imu_link">
         <visual>
             <geometry>
@@ -80,5 +81,5 @@
     </link>
     <!--sensor ultrasonico-->
-    <link name = "range_link">
+    <link name = "${tf_prefix}range_link">
         <visual>
             <geometry>
@@ -95,38 +96,38 @@
         Ubicación Justo debajo del chasis, a altura de las ruedas
     -->
-    <joint name="base_joint" type="fixed">
-        <parent link="base_footprint"/>
-        <child link="base_link"/>
+    <joint name="${tf_prefix}base_joint" type="fixed">
+        <parent link="${tf_prefix}base_footprint"/>
+        <child link="${tf_prefix}base_link"/>
         <origin xyz="0 0 0.01" rpy="0 0 0"/> <!--${wheel_radius}-->
     </joint>
-    <joint name="base_right_wheel_joint" type="continuous">
-        <parent link="base_link"/>
-        <child link="right_wheel_link"/>
+    <joint name="${tf_prefix}base_right_wheel_joint" type="continuous">
+        <parent link="${tf_prefix}base_link"/>
+        <child link="${tf_prefix}right_wheel_link"/>
         <origin xyz="-0.023 -0.09 0.03" rpy="0 0 0"/>
         <axis xyz="0 1 0"/>
-        <limit velocity="16.5" effort="2.5"/>
+        <limit velocity="4.5" effort="2.5"/>
     </joint>
-    <joint name="base_left_wheel_joint" type="continuous">
-        <parent link="base_link"/>
-        <child link="left_wheel_link"/>
+    <joint name="${tf_prefix}base_left_wheel_joint" type="continuous">
+        <parent link="${tf_prefix}base_link"/>
+        <child link="${tf_prefix}left_wheel_link"/>
         <origin xyz="-0.023 0.09 0.03" rpy="0 0 0"/>
         <axis xyz="0 1 0"/>
-        <limit velocity="16.5" effort="2.5"/>
+        <limit velocity="4.5" effort="2.5"/>
     </joint> <!--Velocidad angular máxima en radianes/segundo Par torsional máximo en Newton-metros (Nm) -->
-    <joint name="base_caster_wheel_joint" type="fixed">
-        <parent link="base_link"/>
-        <child link="caster_wheel_link"/>
+    <joint name="${tf_prefix}base_caster_wheel_joint" type="fixed">
+        <parent link="${tf_prefix}base_link"/>
+        <child link="${tf_prefix}caster_wheel_link"/>
         <origin xyz="0.09 0 0" rpy="0 0 0"/>
     </joint>
     <!-- Joint between base_link and imu_link -->
-    <joint name="imu_joint" type="fixed">
-        <parent link="base_link"/>
-        <child link="imu_link"/>
+    <joint name="${tf_prefix}imu_joint" type="fixed">
+        <parent link="${tf_prefix}base_link"/>
+        <child link="${tf_prefix}imu_link"/>
         <origin xyz="-0.06 -0.0675 ${base_height + 0.0035}" rpy="0 0 0"/>
     </joint>
     <!-- Joint between base_link and imu_link -->
-    <joint name="range_joint" type="fixed">
-        <parent link="base_link"/>
-        <child link="range_link"/>
+    <joint name="${tf_prefix}range_joint" type="fixed">
+        <parent link="${tf_prefix}base_link"/>
+        <child link="${tf_prefix}range_link"/>
         <origin xyz="${base_length/2} 0 ${wheel_radius}" rpy="0 0 0"/>
     </joint>

File: src/diffdrive_description/urdf/my_robot.urdf.xacro (robot description, xacro)
@@ -1,5 +1,8 @@
 <?xml version="1.0"?>
 <robot name="Nav2bot" xmlns:xacro="http://www.ros.org/wiki/xacro">
-    <xacro:include filename="common_properties.xacro"/>
-    <xacro:include filename="mobile_base.xacro"/>
+    <!-- Define el tf_prefix para este robot -->
+    <xacro:property name="tf_prefix" value=""/>
+    <!-- Incluye propiedades y base -->
+    <xacro:include filename="$(find diffdrive_description)/urdf/common_properties.xacro"/>
+    <xacro:include filename="$(find diffdrive_description)/urdf/mobile_base.xacro"/>
 </robot>
